Commit message: Actualizacion final del robot RRR y trayectoria ROS2 con un punto y coordenadas

File: ros/robot_ws/src/robot_description/urdf/robot_rrr.urdf (robot description, URDF)
Before this commit: robot robot, 4 links, 3 joints
Links:
- removed link arm_link
- removed link forearm_link
- removed link shoulder_link
- added link column_link; visual cylinder length=0.50 radius=0.055
- added link elbow_disk_link; visual cylinder length=0.08 radius=0.065
- added link end_effector; visual sphere radius=0.055
- added link link1; visual box size=0.60 0.06 0.06
- added link link2; visual box size=0.60 0.06 0.06
- added link rotating_base_link; visual cylinder length=0.08 radius=0.24
- added link shoulder_disk_link; visual cylinder length=0.08 radius=0.075
- added link world
- link base_link: geometry visual cylinder length=0.10 radius=0.28
Joints:
- removed joint arm_joint
- removed joint forearm_joint
- removed joint shoulder_joint
- added joint base_joint: type revolute, parent base_link, child rotating_base_link, origin xyz=0 0 0.08 rpy=0 0 0, axis 0 0 1, limit lower=-3.1416 upper=3.1416 effort=20 velocity=2
- added joint column_joint: type fixed, parent rotating_base_link, child column_link, origin xyz=0 0 0.15 rpy=0 0 0
- added joint elbow_disk_joint: type fixed, parent link1, child elbow_disk_link, origin xyz=0.60 0 0 rpy=0 0 0
- added joint end_effector_joint: type fixed, parent link2, child end_effector, origin xyz=0.60 0 0 rpy=0 0 0
- added joint joint1: type revolute, parent shoulder_disk_link, child link1, origin xyz=0 0 0 rpy=0 0 0, axis 0 1 0, limit lower=-3.1416 upper=3.1416 effort=20 velocity=2
- added joint joint2: type revolute, parent elbow_disk_link, child link2, origin xyz=0 0 0 rpy=0 0 0, axis 0 1 0, limit lower=-3.1416 upper=3.1416 effort=20 velocity=2
- added joint shoulder_disk_joint: type fixed, parent column_link, child shoulder_disk_link, origin xyz=0 0 0.52 rpy=0 0 0
- added joint world_to_base: type fixed, parent world, child base_link, origin xyz=0 0 0 rpy=0 0 0
